File: tools/pisa/pisa/pisa.kicad_sch (KiCad schematic)
At the start: 15 parts, among them J1 Bus_ISA_8bit, J2 Raspberry_Pi_2_3, J3 DIN-5_180degree, J4 Conn_02x06_Odd_Even, U1 LM7905_TO220, U2 74LVC245A, U3 74LS245, U4 74LS245, U5 74LS245, U6 LM1117T-3.3

Commit message: Updeated ISA board
Parts:
- added U7: 74LS245, symbol 74xx:74LS245
- added X1: ACO-14.31818MHz, Oscillator:Oscillator_DIP-14, symbol Oscillator:ACO-xxxMHz
- U2: value 74LVC245A -> 74LVC245
- U3: value 74LS245 -> 74LVC245
Connections:
- net +3.3V: now also U3.20 (VCC), U5.20 (VCC)
- net +5V: now also U2.20 (VCC), U4.20 (VCC), U7.20 (VCC), X1.14 (Vcc)
- net A0: now also U7.2 (A0)
- net A1: now also U7.3 (A1)
- net A10: now also U4.4 (A2)
- net A11: now also U4.5 (A3)
- net A2: now also U7.4 (A2)
- net A3: now also U7.5 (A3)
- net A4: now also U7.6 (A4)
- net A5: now also U7.7 (A5)
- net A6: now also U7.8 (A6)
- net A7: now also U7.9 (A7)
- net A8: now also U4.2 (A0)
- net A9: now also U4.3 (A1)
- net D0: now also U2.2 (A0), U3.18 (B0)
- net D1: now also U2.3 (A1), U3.17 (B1)
- net D2: now also U2.4 (A2), U3.16 (B2)
- net D3: now also U2.5 (A3), U3.15 (B3)
- net D4: now also U2.6 (A4), U3.14 (B4)
- net D5: now also U2.7 (A5), U3.13 (B5)
- net D6: now also U2.8 (A6), U3.12 (B6)
- net D7: now also U2.9 (A7), U3.11 (B7)
- net GND: now also J1.27 (TC), J1.28 (ALE), U2.1 (A->B), U2.10 (GND), U3.1 (A->B), U3.10 (GND), U4.1 (A->B), U4.10 (GND), U4.19 (CE), U5.1 (A->B), U5.10 (GND), U5.11 (B7), U5.12 (B6), U5.13 (B5), U5.14 (B4), U5.15 (B3), U5.19 (CE), U7.1 (A->B), U7.10 (GND), U7.19 (CE), X1.7 (GND)
- net IO_REDY: now also U5.17 (B1)
- net IRQ: now also U5.16 (B2)
- net D7_LV: now reaches U2.11 (B7)
- net D7_LV: now also J2.35 (GPIO19/MISO1), U3.9 (A7)
- net D6_LV: now reaches U2.12 (B6)
- net D6_LV: now also J2.12 (GPIO18/PWM0), U3.8 (A6)
- net D5_LV: now reaches U2.13 (B5)
- net D5_LV: now also J2.11 (GPIO17), U3.7 (A5)
- net D4_LV: now reaches U2.14 (B4)
- net D4_LV: now also J2.36 (GPIO16), U3.6 (A4)
- net D3_LV: now reaches U2.15 (B3)
- net D3_LV: now also J2.10 (GPIO15/RXD), U3.5 (A3)
- net D2_LV: now reaches U2.16 (B2)
- net D2_LV: now also J2.8 (GPIO14/TXD), U3.4 (A2)
- net D1_LV: now reaches U2.17 (B1)
- net D1_LV: now also J2.33 (PWM1/GPIO13), U3.3 (A1)
- net D0_LV: now reaches U2.18 (B0)
- net D0_LV: now also J2.32 (PWM0/GPIO12), U3.2 (A0)
- net IOW: now reaches U2.19 (CE)
- net IOW: now also J1.13 (~{IOW}), U4.7 (A5)
- net IOR_LV: now reaches U3.19 (CE)
- net IOR_LV: now also J2.15 (GPIO22), U4.12 (B6)
- net CLK_LV: now reaches U4.11 (B7)
- net CLK_LV: now also J2.16 (GPIO23), J2.38 (GPIO20/MOSI1), U4.14 (B4)
- net IOW_LV: now reaches U4.13 (B5)
- net IOW_LV: now also J2.40 (GPIO21/SCLK1)
- net A11_LV: now reaches U4.15 (B3)
- net A11_LV: now also J2.23 (SCLK0/GPIO11)
- net A10_LV: now reaches U4.16 (B2)
- net A10_LV: now also J2.19 (MOSI0/GPIO10)
- net A9_LV: now reaches U4.17 (B1)
- net A9_LV: now also J2.21 (MISO0/GPIO9)
- net A8_LV: now reaches U4.18 (B0)
- net A8_LV: now also J2.24 (~{CE0}/GPIO8)
- net CLK: now reaches U4.6 (A4)
- net CLK: now also J1.2 (RESET), J1.20 (CLK), U4.9 (A7)
- net IOR: now reaches U4.8 (A6)
- net IOR: now also J1.14 (~{IOR})
- net IRQ_LV: now reaches J2.18 (GPIO24)
- net IRQ_LV: now also U5.4 (A2)
- net IO_REDY_LV: now reaches J2.22 (GPIO25)
- net IO_REDY_LV: now also U5.3 (A1)
- net A7_LV: now reaches J2.26 (~{CE1}/GPIO7)
- net A7_LV: now also U7.11 (B7)
- net A0_LV: now reaches J2.27 (ID_SD/GPIO0)
- net A0_LV: now also U7.18 (B0)
- net A1_LV: now reaches J2.28 (ID_SC/GPIO1)
- net A1_LV: now also U7.17 (B1)
- net A5_LV: now reaches J2.29 (GCLK1/GPIO5)
- net A5_LV: now also U7.13 (B5)
- net A2_LV: now reaches J2.3 (SDA/GPIO2)
- net A2_LV: now also U7.16 (B2)
- net A6_LV: now reaches J2.31 (GCLK2/GPIO6)
- net A6_LV: now also U7.12 (B6)
- net IO_CHECK_LV: now reaches J2.37 (GPIO26)
- net IO_CHECK_LV: now also U5.2 (A0)
- net A3_LV: now reaches J2.5 (SCL/GPIO3)
- net A3_LV: now also U7.15 (B3)
- net A4_LV: now reaches J2.7 (GCLK0/GPIO4)
- net A4_LV: now also U7.14 (B4)
- net at J1.30 (OSC): now also X1.8 (OUT)
- net IO_CHECK: now reaches J1.32 (IO)
- net IO_CHECK: now also U5.18 (B0)
- no-connect marks 7 -> 12
Other:
- title: (none) -> PiISA
- moved on the sheet: C1, C2, C3, C4, J2, J3, U1, U2, U3, U4, U5, U6

Commit message: Fixed some bugs.
Parts:
- removed J1: Bus_ISA_8bit, symbol Connector:Bus_ISA_8bit
- removed J4: Conn_02x06_Odd_Even, symbol Connector_Generic:Conn_02x06_Odd_Even
- added C5, C6, C7, C8, C9: C_Small, symbol Device:C_Small
- added J1: Bus_ISA_Socket_8bit, symbol bus_isa_socket_8bit:Bus_ISA_Socket_8bit
- added J4: Conn_01x02, symbol Connector_Generic:Conn_01x02
- added SW1: SW_DIP_x04, symbol Switch:SW_DIP_x04
- U4, U5, U7: value 74LS245 -> 74LVC245
Connections:
- net IO_CHECK is gone; now on net IO_REDY: U5.18 (B0)
- net IRQ is gone; now on net IRQ5: U5.16 (B2)
- net +12V: now also J1.9 (+12V)
- net +3.3V: now also C8.1, C9.1
- net +5V: now also C5.2, C6.2, C7.2, J1.11 (~{SMEMW}), J1.12 (~{SMEMR}), J1.15 (~{DACK3}), J1.17 (~{DACK1}), J1.26 (~{DACK2}), J1.29 (VCC), J1.3 (VCC), J4.2 (Pin_2); no longer J2.2 (5V), J2.4 (5V)
- net -12V: now also J1.7 (-12V)
- net -5V: now also J1.5 (-5V)
- net A0: now also J1.62 (BA00)
- net A1: now also J1.61 (BA01)
- net A10: now also J1.52 (BA10)
- net A11: now also J1.51 (BA11)
- net A2: now also J1.60 (BA02)
- net A3: now also J1.59 (BA03)
- net A4: now also J1.58 (BA04)
- net A5: now also J1.57 (BA05)
- net A6: now also J1.56 (BA06)
- net A7: now also J1.55 (BA07)
- net A8: now also J1.54 (BA08)
- net A9: now also J1.53 (BA09)
- net CLK: now also J1.20 (CLK); no longer U4.9 (A7)
- net CLK_LV: no longer J2.16 (GPIO23), U4.11 (B7)
- net D0: now also J1.40 (DB0)
- net D1: now also J1.39 (DB1)
- net D2: now also J1.38 (DB2)
- net D3: now also J1.37 (DB3)
- net D4: now also J1.36 (DB4)
- net D5: now also J1.35 (DB5)
- net D6: now also J1.34 (DB6)
- net D7: now also J1.33 (DB7)
- net GND: now also C5.1, C6.1, C7.1, C8.2, C9.2, J1.1 (GND), J1.10 (GND), J1.27 (TC), J1.28 (ALE), J1.31 (GND), J1.42 (AEN), J1.43 (BA19), J1.44 (BA18), J1.45 (BA17), J1.46 (BA16), J1.47 (BA15), J1.48 (BA14), J1.49 (BA13), J1.50 (BA12); no longer U5.11 (B7), U5.12 (B6), U5.13 (B5), U5.14 (B4), U5.15 (B3)
- net IOR: now also J1.14 (~{IOR})
- net IOW: now also J1.13 (~{IOW})
- net IO_REDY: now also J1.41 (IO_READY); no longer U5.17 (B1)
- net IO_REDY_LV: now also J2.13 (GPIO27), U5.2 (A0); no longer J2.22 (GPIO25), U5.3 (A1)
- net IRQ2: now also J1.4 (IRQ2), SW1.8
- net IRQ3: now also U5.11 (B7), U5.12 (B6), U5.13 (B5), U5.14 (B4), U5.15 (B3), J1.25 (IRQ3)
- net IRQ4: now also J1.24 (IRQ4), SW1.7
- net IRQ5: now also J1.23 (IRQ5)
- net IRQ6: now also J1.22 (IRQ6), SW1.6
- net IRQ7: now also J1.21 (IRQ7), SW1.5
- net at R1.2: now also J1.19 (~{DACK0})
- net at X1.8 (OUT): now also J1.30 (OSC)
- net IRQ3_LV: now reaches U5.5 (A3)
- net IRQ3_LV: now also J2.18 (GPIO24)
- net IO_CHECK_LV renamed IRQX_LV
- net IRQX_LV: now also U5.3 (A1); no longer U5.2 (A0)
- net IRQ_LV renamed IRQ5_LV
- net IRQ5_LV: now also J2.22 (GPIO25); no longer J2.18 (GPIO24)
- new net: J2.2 (5V), J2.4 (5V), J4.1 (Pin_1)
- new net IRQX: SW1.1, SW1.2, SW1.3, SW1.4, U5.17 (B1)
- new net RESET: J1.2 (RESET), U4.9 (A7)
- new net RESET_LV: J2.16 (GPIO23), U4.11 (B7)
- no-connect marks 12 -> 11
Other:
- company: (none) -> Copyright (c) 2023 Andreas T Jonsson

Commit message: Minor update
Parts:
- C5, C6, C7, C8, C9: value C_Small -> 0.1uF
Changed lines of the file:
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@@
       (effects (font (size 1.27 1.27)))
     )
-    (property "Value" "C_Small" (at 129.5463 22.86 90)
+    (property "Value" "0.1uF" (at 129.5463 22.86 90)
       (effects (font (size 1.27 1.27)))
     )
@@
       (effects (font (size 1.27 1.27)))
     )
-    (property "Value" "C_Small" (at 139.7063 31.75 90)
+    (property "Value" "0.1uF" (at 139.7063 31.75 90)
       (effects (font (size 1.27 1.27)))
     )
@@
       (effects (font (size 1.27 1.27)))
     )
-    (property "Value" "C_Small" (at 139.7063 22.86 90)
+    (property "Value" "0.1uF" (at 139.7063 22.86 90)
       (effects (font (size 1.27 1.27)))
     )
@@
       (effects (font (size 1.27 1.27)))
     )
-    (property "Value" "C_Small" (at 129.5463 31.75 90)
+    (property "Value" "0.1uF" (at 129.5463 31.75 90)
       (effects (font (size 1.27 1.27)))
     )
@@
       (effects (font (size 1.27 1.27)))
     )
-    (property "Value" "C_Small" (at 139.7063 40.64 90)
-      (effects (font (size 1.27 1.27)))
-    )
+    (property "Value" "0.1uF" (at 139.7063 40.64 90)
+      (effects (font (size 1.27 1.27)))
+    )
